Commit message: Adapted to tf of Ting's omni

File: urdf/omni.urdf (robot description, URDF)
Before this commit: robot omni_bot, 3 links, 2 joints
Joints:
- joint base_link_to_imu: origin xyz=0.06 0.02 0.0 rpy=0.0 0.0 0.69 -> xyz=-0.005 0.035 -0.06 rpy=3.1415926 0.0 3.1415926
- joint base_link_to_laser: origin xyz=0.0 0.0 0.235 rpy=0.0 0.0 3.14 -> xyz=0.0 0.0 0.125 rpy=0.0 0.0 3.1415926

Commit message: Adatped Kubot to ROS2

File: urdf/omni.urdf (robot description, URDF)
Before this commit: robot omni_bot, 3 links, 2 joints
Links:
- removed link base_imu
- added link base_footprint
- added link imu_link
- link base_link: mass None -> 6.000; geometry collision box size=0.33 0.33 0.32; visual mesh filename=package://omni_ros2/meshes/apollo/base_link.stl scale=1 1 1
- link laser_frame: mass None -> 0.17934; geometry collision cylinder length=0.0315 radius=0.035; visual mesh filename=package://omni_ros2/meshes/apollo/laser_link.stl scale=1 1 1
Joints:
- removed joint base_link_to_imu
- removed joint base_link_to_laser
- added joint base_joint: type fixed, parent base_footprint, child base_link, origin xyz=0 0 0 rpy=0 0 0
- added joint imu_joint: type fixed, parent base_link, child imu_link, origin xyz=0 0 0.11 rpy=0 0 0
- added joint laser_joint: type fixed, parent base_link, child laser_frame, origin xyz=0.11 0 0.31 rpy=0 0 3.14
