Commit message: First version Kubot_ros2

File: urdf/omni_bot.urdf (robot description, URDF)
Before this commit: robot omni_bot, 4 links, 3 joints
Links:
- removed link base_footprint
- link base_link: mass 6.000 -> None; geometry collision box size=0.33 0.33 0.32; visual mesh filename=package://omni_ros2/meshes/apollo/base_link.stl
- link laser_frame: geometry collision cylinder length=0.0315 radius=0.035; visual mesh filename=package://omni_ros2/meshes/apollo/laser_link.stl
Joints:
- removed joint base_joint
